Commit message: add Readme

File: src/husky_description/urdf/accessories/vlp16_mount.urdf.xacro (robot description, xacro)
@@ -2,5 +2,5 @@
 <robot xmlns:xacro="http://wiki.ros.org/xacro">
   <xacro:include filename="$(find velodyne_description)/urdf/VLP-16.urdf.xacro" />
-  <xacro:macro name="vlp16_mount" params="prefix parent_link topic height:=0.12 *origin">
+  <xacro:macro name="vlp16_mount" params="prefix parent_link topic height:=0.08 *origin">
     <!--
       The VLP16 is mounted to a pair of extrusion rods on top of the main sensor arch
@@ -15,5 +15,5 @@
           <color rgba="1 1 1 1" />
         </material>
-        <origin xyz="0 0 0.00315" rpy="0 0 0" />
+        <origin xyz="0.1 0 0.00315" rpy="0 0 0" />
       </visual>
       <collision>
@@ -21,5 +21,5 @@
           <box size="0.04 0.02 ${height}" />
         </geometry>
-        <origin xyz="0 0 0" rpy="0 0 0" />
+        <origin xyz="0.1 0 0" rpy="0 0 0" />
       </collision>
     </link>
@@ -28,9 +28,10 @@
         <geometry>
           <box size="0.04 0.02 ${height}" />
+          <!-- <box size="0.04 0.02 0.07" /> -->
         </geometry>
         <material name="black">
           <color rgba="1 1 1 1" />
         </material>
-        <origin xyz="0 0 0" rpy="0 0 0" />
+        <origin xyz="0.1 0 0" rpy="0 0 0" />
       </visual>
       <collision>
@@ -38,5 +39,5 @@
           <box size="0.04 0.02 ${height}" />
         </geometry>
-        <origin xyz="0 0 0" rpy="0 0 0" />
+        <origin xyz="0.1 0 0" rpy="0 0 0" />
       </collision>
     </link>
@@ -49,5 +50,5 @@
           <color rgba="1 1 1 1" />
         </material>
-        <origin xyz="0 0 0" rpy="0 0 0" />
+        <origin xyz="0.1 0 0" rpy="0 0 0" />
       </visual>
       <collision>
@@ -55,5 +56,5 @@
           <box size="0.04 0.02 ${height}" />
         </geometry>
-        <origin xyz="0 0 0" rpy="0 0 0" />
+        <origin xyz="0.1 0 0" rpy="0 0 0" />
       </collision>
     </link>
@@ -66,18 +67,18 @@
       <parent link="${prefix}vlp16_mount_base_link" />
       <child link="${prefix}vlp16_mount_left_support" />
-      <origin xyz="0 0.06 ${height/2}" rpy="0 0 0"/>
+      <origin xyz="0.1 0.06 ${height/2}" rpy="0 0 0"/>
     </joint>
     <joint name="${prefix}vlp16_mount_right_support_joint" type="fixed">
       <parent link="${prefix}vlp16_mount_base_link" />
       <child link="${prefix}vlp16_mount_right_support" />
-      <origin xyz="0 -0.06 ${height/2}" rpy="0 0 0"/>
+      <origin xyz="0.1 -0.06 ${height/2}" rpy="0 0 0"/>
     </joint>
     <joint name="${prefix}vlp16_mount_plate_joint" type="fixed">
       <parent link="${prefix}vlp16_mount_base_link" />
       <child link="${prefix}vlp16_mount_plate" />
-      <origin xyz="0 0 ${height}" rpy="0 0 0"/>
+      <origin xyz="0.1 0 ${height}" rpy="0 0 0"/>
     </joint>
     <xacro:VLP-16 parent="${prefix}vlp16_mount_plate" topic="${topic}" name="${prefix}velodyne">
-      <origin xyz="0 0 0.0063" rpy="0 0 0" />
+      <origin xyz="0.1 0 0.0063" rpy="0 0 0" />
     </xacro:VLP-16>
   </xacro:macro>

File: src/husky_description/urdf/husky.urdf.xacro (robot description, xacro)
@@ -23,5 +23,5 @@
 <robot name="husky" xmlns:xacro="http://ros.org/wiki/xacro">
   <!-- IMU Link -->
-  <xacro:arg name="imu_xyz"     default="$(optenv HUSKY_IMU_XYZ 0.19 0 0.149)"/>
+  <xacro:arg name="imu_xyz"     default="$(optenv HUSKY_IMU_XYZ 0.28 0 0.2)"/>
   <xacro:arg name="imu_rpy"     default="$(optenv HUSKY_IMU_RPY 0 0 0)"/>
   <xacro:arg name="imu_parent"  default="$(optenv HUSKY_IMU_PARENT base_link)"/>
